File: LowPassFilter.sch (KiCad schematic (older format))
At the start: 38 parts, among them U43 ADA4625, U44 OPA2189, U45 ADA4625, U46 ADA4625, U47 OPA2189, U48 ADA4625, U49 ADA4625, U50 ADA4625, U51 ADA4625, U52 ADA4625

Commit message: Add files via upload
Updated opamps to ada4522 because they have lower bias current.
Parts:
- removed R88, R91, R94, R97: 33R, symbol R
- removed U44, U47: OPA2189, symbol TLC272
Other:
- note added: "Low pass filter; 150nv/sqrt(8) ==>\n0.1-10Hz noise = 53 nV p-p (typical)"
Changed lines of the file:
@@
 $Descr A4 11693 8268
 encoding utf-8
-Sheet 7 5
+Sheet 4 6
 Title "DIY Differential Voltmeter.  Version 1"
 Date "2019-05-20"
@@
 NoConn ~ 2000 2500
 $Comp
-L +15V #PWR100
+L +15V #PWR082
 U 1 1 5C72FAC2
 P 1900 1900
-F 0 "#PWR100" H 1900 1750 50  0001 C CNN
+F 0 "#PWR082" H 1900 1750 50  0001 C CNN
 F 1 "+15V" H 1900 2040 50  0000 C CNN
 F 2 "" H 1900 1900 50  0001 C CNN
@@
 NoConn ~ 2000 3450
 $Comp
-L +15V #PWR103
+L +15V #PWR083
 U 1 1 5C72FB96
 P 1900 2850
-F 0 "#PWR103" H 1900 2700 50  0001 C CNN
+F 0 "#PWR083" H 1900 2700 50  0001 C CNN
 F 1 "+15V" H 1900 2990 50  0000 C CNN
 F 2 "" H 1900 2850 50  0001 C CNN
@@
 NoConn ~ 2000 4400
 $Comp
-L +15V #PWR106
+L +15V #PWR084
 U 1 1 5C72FD4C
 P 1900 3800
-F 0 "#PWR106" H 1900 3650 50  0001 C CNN
+F 0 "#PWR084" H 1900 3650 50  0001 C CNN
 F 1 "+15V" H 1900 3940 50  0000 C CNN
 F 2 "" H 1900 3800 50  0001 C CNN
@@
 NoConn ~ 2000 5350
 $Comp
-L +15V #PWR109
+L +15V #PWR085
 U 1 1 5C72FD6A
 P 1900 4750
-F 0 "#PWR109" H 1900 4600 50  0001 C CNN
+F 0 "#PWR085" H 1900 4600 50  0001 C CNN
 F 1 "+15V" H 1900 4890 50  0000 C CNN
 F 2 "" H 1900 4750 50  0001 C CNN
@@
 NoConn ~ 4800 2600
 $Comp
-L +15V #PWR110
+L +15V #PWR086
 U 1 1 5C7303F3
 P 4700 2000
-F 0 "#PWR110" H 4700 1850 50  0001 C CNN
+F 0 "#PWR086" H 4700 1850 50  0001 C CNN
 F 1 "+15V" H 4700 2140 50  0000 C CNN
 F 2 "" H 4700 2000 50  0001 C CNN
@@
 NoConn ~ 4800 3550
 $Comp
-L +15V #PWR115
+L +15V #PWR087
 U 1 1 5C730411
 P 4700 2950
-F 0 "#PWR115" H 4700 2800 50  0001 C CNN
+F 0 "#PWR087" H 4700 2800 50  0001 C CNN
 F 1 "+15V" H 4700 3090 50  0000 C CNN
 F 2 "" H 4700 2950 50  0001 C CNN
@@
 NoConn ~ 4800 4500
 $Comp
-L +15V #PWR118
+L +15V #PWR088
 U 1 1 5C730433
 P 4700 3900
-F 0 "#PWR118" H 4700 3750 50  0001 C CNN
+F 0 "#PWR088" H 4700 3750 50  0001 C CNN
 F 1 "+15V" H 4700 4040 50  0000 C CNN
 F 2 "" H 4700 3900 50  0001 C CNN
@@
 NoConn ~ 4800 5450
 $Comp
-L +15V #PWR121
+L +15V #PWR089
 U 1 1 5C730451
 P 4700 4850
-F 0 "#PWR121" H 4700 4700 50  0001 C CNN
+F 0 "#PWR089" H 4700 4700 50  0001 C CNN
 F 1 "+15V" H 4700 4990 50  0000 C CNN
 F 2 "" H 4700 4850 50  0001 C CNN
@@
 $EndComp
 $Comp
-L GNDA #PWR104
+L GNDA #PWR090
 U 1 1 5C7314D4
 P 1400 3350
-F 0 "#PWR104" H 1400 3100 50  0001 C CNN
+F 0 "#PWR090" H 1400 3100 50  0001 C CNN
 F 1 "GNDA" H 1400 3200 50  0000 C CNN
 F 2 "" H 1400 3350 50  0001 C CNN
@@
 	1    1400 3350
 	1    0    0    -1
-$EndComp
-$Comp
-L TLC272 U44
-U 2 1 5C73813C
-P 10350 2900
-F 0 "U44" H 10350 3100 50  0000 L CNN
-F 1 "OPA2189" H 10350 2700 50  0000 L CNN
-F 2 "" H 10350 2900 50  0001 C CNN
-F 3 "" H 10350 2900 50  0001 C CNN
-	2    10350 2900
-	1    0    0    -1
-$EndComp
-$Comp
-L R R91
-U 1 1 5C7383DD
-P 10800 2900
-F 0 "R91" V 10880 2900 50  0000 C CNN
-F 1 "33R" V 10800 2900 50  0000 C CNN
-F 2 "" V 10730 2900 50  0001 C CNN
-F 3 "" H 10800 2900 50  0001 C CNN
-	1    10800 2900
-	0    1    1    0
-$EndComp
-$Comp
-L TLC272 U44
-U 1 1 5C7386D2
-P 10350 2100
-F 0 "U44" H 10350 2300 50  0000 L CNN
-F 1 "OPA2189" H 10350 1900 50  0000 L CNN
-F 2 "" H 10350 2100 50  0001 C CNN
-F 3 "" H 10350 2100 50  0001 C CNN
-	1    10350 2100
-	1    0    0    -1
-$EndComp
-$Comp
-L R R88
-U 1 1 5C7386D8
-P 10800 2100
-F 0 "R88" V 10880 2100 50  0000 C CNN
-F 1 "33R" V 10800 2100 50  0000 C CNN
-F 2 "" V 10730 2100 50  0001 C CNN
-F 3 "" H 10800 2100 50  0001 C CNN
-	1    10800 2100
-	0    1    1    0
-$EndComp
-$Comp
-L TLC272 U47
-U 2 1 5C7389AC
-P 10350 4500
-F 0 "U47" H 10350 4700 50  0000 L CNN
-F 1 "OPA2189" H 10350 4300 50  0000 L CNN
-F 2 "" H 10350 4500 50  0001 C CNN
-F 3 "" H 10350 4500 50  0001 C CNN
-	2    10350 4500
-	1    0    0    -1
-$EndComp
-$Comp
-L R R97
-U 1 1 5C7389B2
-P 10800 4500
-F 0 "R97" V 10880 4500 50  0000 C CNN
-F 1 "33R" V 10800 4500 50  0000 C CNN
-F 2 "" V 10730 4500 50  0001 C CNN
-F 3 "" H 10800 4500 50  0001 C CNN
-	1    10800 4500
-	0    1    1    0
-$EndComp
-$Comp
-L TLC272 U47
-U 1 1 5C7389BC
-P 10350 3700
-F 0 "U47" H 10350 3900 50  0000 L CNN
-F 1 "OPA2189" H 10350 3500 50  0000 L CNN
-F 2 "" H 10350 3700 50  0001 C CNN
-F 3 "" H 10350 3700 50  0001 C CNN
-	1    10350 3700
-	1    0    0    -1
-$EndComp
-$Comp
-L R R94
-U 1 1 5C7389C2
-P 10800 3700
-F 0 "R94" V 10880 3700 50  0000 C CNN
-F 1 "33R" V 10800 3700 50  0000 C CNN
-F 2 "" V 10730 3700 50  0001 C CNN
-F 3 "" H 10800 3700 50  0001 C CNN
-	1    10800 3700
-	0    1    1    0
 $EndComp
 $Comp
@@
 $EndComp
 $Comp
-L GNDA #PWR101
+L GNDA #PWR091
 U 1 1 5C859F96
 P 1400 2400
-F 0 "#PWR101" H 1400 2150 50  0001 C CNN
+F 0 "#PWR091" H 1400 2150 50  0001 C CNN
 F 1 "GNDA" H 1400 2250 50  0000 C CNN
 F 2 "" H 1400 2400 50  0001 C CNN
@@
 $EndComp
 $Comp
-L GNDA #PWR107
+L GNDA #PWR092
 U 1 1 5C85A060
 P 1400 4300
-F 0 "#PWR107" H 1400 4050 50  0001 C CNN
+F 0 "#PWR092" H 1400 4050 50  0001 C CNN
 F 1 "GNDA" H 1400 4150 50  0000 C CNN
 F 2 "" H 1400 4300 50  0001 C CNN
@@
 Connection ~ 5400 2300
 Connection ~ 1400 3050
-Wire Wire Line
-	10050 3000 10050 3350
-Wire Wire Line
-	10050 3350 10650 3350
-Wire Wire Line
-	10650 3350 10650 2900
-Connection ~ 10650 2900
-Wire Wire Line
-	10050 2200 10050 2550
-Wire Wire Line
-	10050 2550 10650 2550
-Wire Wire Line
-	10650 2550 10650 2100
-Connection ~ 10650 2100
-Wire Wire Line
-	10050 4600 10050 4950
-Wire Wire Line
-	10050 4950 10650 4950
-Wire Wire Line
-	10650 4950 10650 4500
-Connection ~ 10650 4500
-Wire Wire Line
-	10050 3800 10050 4150
-Wire Wire Line
-	10050 4150 10650 4150
-Wire Wire Line
-	10650 4150 10650 3700
-Connection ~ 10650 3700
-Wire Wire Line
-	10050 2000 9800 2000
-Wire Wire Line
-	9800 2000 9800 4400
-Wire Wire Line
-	9800 4400 10050 4400
-Wire Wire Line
-	10050 3600 9800 3600
-Connection ~ 9800 3600
-Wire Wire Line
-	10050 2800 9800 2800
-Connection ~ 9800 2800
-Wire Wire Line
-	10950 2100 10950 4500
 Connection ~ 1400 2100
 Connection ~ 1400 4000
@@
 $EndComp
 $Comp
-L GNDA #PWR111
+L GNDA #PWR093
 U 1 1 5C85BD8B
 P 1400 5250
-F 0 "#PWR111" H 1400 5000 50  0001 C CNN
+F 0 "#PWR093" H 1400 5000 50  0001 C CNN
 F 1 "GNDA" H 1400 5100 50  0000 C CNN
 F 2 "" H 1400 5250 50  0001 C CNN
@@
 $EndComp
 $Comp
-L GNDA #PWR114
+L GNDA #PWR094
 U 1 1 5C85C456
 P 4000 2850
-F 0 "#PWR114" H 4000 2600 50  0001 C CNN
+F 0 "#PWR094" H 4000 2600 50  0001 C CNN
 F 1 "GNDA" H 4000 2700 50  0000 C CNN
 F 2 "" H 4000 2850 50  0001 C CNN
@@
 $EndComp
 $Comp
-L GNDA #PWR116
+L GNDA #PWR095
 U 1 1 5C85C502
 P 4000 3450
-F 0 "#PWR116" H 4000 3200 50  0001 C CNN
+F 0 "#PWR095" H 4000 3200 50  0001 C CNN
 F 1 "GNDA" H 4000 3300 50  0000 C CNN
 F 2 "" H 4000 3450 50  0001 C CNN
@@
 $EndComp
 $Comp
-L GNDA #PWR119
+L GNDA #PWR096
 U 1 1 5C85C648
 P 4000 4400
-F 0 "#PWR119" H 4000 4150 50  0001 C CNN
+F 0 "#PWR096" H 4000 4150 50  0001 C CNN
 F 1 "GNDA" H 4000 4250 50  0000 C CNN
 F 2 "" H 4000 4400 50  0001 C CNN
@@
 $EndComp
 $Comp
-L GNDA #PWR122
+L GNDA #PWR097
 U 1 1 5C85D204
 P 4000 5350
-F 0 "#PWR122" H 4000 5100 50  0001 C CNN
+F 0 "#PWR097" H 4000 5100 50  0001 C CNN
 F 1 "GNDA" H 4000 5200 50  0000 C CNN
 F 2 "" H 4000 5350 50  0001 C CNN
@@
 	1700 4000 1400 4000
 Connection ~ 1100 4950
-Text GLabel 9800 2800 0    60   Input ~ 0
-BufferIn
-Text GLabel 10950 2900 2    60   Input ~ 0
-BufferOut
-Connection ~ 10950 3700
-Connection ~ 10950 2900
 Text GLabel 3700 3150 0    60   Input ~ 0
 DacOut
@@
 Wire Wire Line
 	5400 2300 5400 5150
+Text Notes 3600 1350 2    60   ~ 0
+Low pass filter; 150nv/sqrt(8) ==>\n0.1-10Hz noise = 53 nV p-p (typical)
 $EndSCHEMATC
